File: Fjernbetjening/Modtager/TocBoatReceiver/TocBoatReceiver.kicad_pcb (KiCad board)
At the start: 2 copper layers, 55 x 85 mm, 40 parts, among them J1 Prog, J2 USB_A, J3 Battery, J4 Conn_01x02, J5 Conn_01x02, J6 SpeedController, J7 Servo, Q1 BC846BS, Q2 AO3400A, Q3 AO3400A, Q4 AO3400A, U1 USBLC6-2SC6, U2 AP1117-33, U6 CP2102N-Axx-xQFN28, U8 ESP32-S2-WROVER

Commit message: mods on PCB done
Parts:
- removed U8: ESP32-S2-WROVER, RF_Module:ESP32-S2-WROVER
- added U3: ESP32-WROOM-32, RF_Module:ESP32-WROOM-32, F.Cu at (140.8, 87.7)
- moved J2 0.41 mm to (137.2, 122.2)
Connections:
- J1 pad 2: +3V3 -> +3.3V
- J1 pad 4: GNDD -> GND
- U1 pad 1: Net-(J2-D-) -> Net-(J2-D+)
- U1 pad 3: Net-(J2-D+) -> Net-(J2-D-)
Routing:
- net D0: track 27.9 -> 53.0 mm, vias 2 -> 4
- net /ESP32/GPIO18: track 3.59 -> 28.4 mm
- net /ESP32/GPIO17: track 4.09 -> 27.8 mm
- net /ESP32/GPIO16: track 30.7 -> 49.2 mm
- net /ESP32/GPIO5: track 37.9 -> 51.0 mm
- net /ESP32/GPIO15: track 7.39 -> 19.5 mm
- net +3.3V: track 106.4 -> 118.0 mm, vias 6 -> 7
- net /ESP32/GPIO14: track 39.6 -> 49.1 mm, vias 2 -> 4
- net GND: track 27.8 -> 26.0 mm, vias 19 -> 51
- net EN: track 43.5 -> 45.1 mm, vias 2 -> 3
- net Net-(J2-D-): track 3.05 -> 4.19 mm
- net Net-(J2-D+): track 3.01 -> 4.12 mm, vias 0 -> 2
- net RX: track 50.5 -> 51.6 mm, vias 0 -> 2
- net TX: track 53.6 -> 52.7 mm, vias 0 -> 2
- added copper zone on F.Cu, net GND
