File: Fjernbetjening/Modtager/TocBoatReceiver/TocBoatReceiver.kicad_sch (KiCad schematic)
At the start: 12 parts, among them J2 USB_A, J3 Battery, J6 SpeedController, J7 Servo, U1 USBLC6-2SC6, U2 AP1117-33

Commit message: mods on PCB done
Connections:
- net at U1.1 (I/O1): now also J2.3 (D+); no longer J2.2 (D-)
- net at U1.3 (I/O2): now also J2.2 (D-); no longer J2.3 (D+)
Other:
- sheet ESP32: file StdEsp32.kicad_sch -> StdEsp32_worm2.kicad_sch
- sheet ESP32 ports: added none; removed GPIO10, GPIO11, GPIO37, GPIO38, GPIO40, GPIO6, GPIO7, GPIO8, GPIO9
Changed lines of the file:
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@@
 	(wire
 		(pts
-			(xy 45.72 93.98) (xy 52.07 93.98)
+			(xy 45.72 93.98) (xy 58.42 93.98)
 		)
 		(stroke
@@
 	(wire
 		(pts
-			(xy 48.26 92.71) (xy 48.26 91.44)
-		)
-		(stroke
-			(width 0)
-			(type default)
-		)
-	)
-	(wire
-		(pts
 			(xy 69.85 123.19) (xy 69.85 127)
 		)
@@
 	(wire
 		(pts
-			(xy 48.26 91.44) (xy 45.72 91.44)
+			(xy 45.72 91.44) (xy 58.42 91.44)
 		)
 		(stroke
@@
 	(wire
 		(pts
-			(xy 58.42 93.98) (xy 58.42 92.71)
-		)
-		(stroke
-			(width 0)
-			(type default)
-		)
-	)
-	(wire
-		(pts
 			(xy 97.79 59.69) (xy 97.79 62.23)
 		)
@@
 	(wire
 		(pts
-			(xy 58.42 92.71) (xy 48.26 92.71)
-		)
-		(stroke
-			(width 0)
-			(type default)
-		)
-	)
-	(wire
-		(pts
 			(xy 69.85 127) (xy 78.74 127)
 		)
@@
 	(wire
 		(pts
-			(xy 52.07 91.44) (xy 58.42 91.44)
-		)
-		(stroke
-			(width 0)
-			(type default)
-		)
-	)
-	(wire
-		(pts
 			(xy 149.86 119.38) (xy 149.86 118.11)
-		)
-		(stroke
-			(width 0)
-			(type default)
-		)
-	)
-	(wire
-		(pts
-			(xy 52.07 93.98) (xy 52.07 91.44)
 		)
 		(stroke
@@
 			)
 		)
-		(property "Sheetfile" "StdEsp32.kicad_sch"
+		(property "Sheetfile" "StdEsp32_worm2.kicad_sch"
 			(at 114.3 141.5546 0)
 			(effects
@@
 			)
 		)
-		(pin "GPIO7" input
-			(at 114.3 115.57 180)
-			(effects
-				(font
-					(size 1.27 1.27)
-				)
-				(justify left)
-			)
-		)
 		(pin "GPIO35" input
 			(at 143.51 99.06 0)
@@
 			)
 		)
-		(pin "GPIO38" input
-			(at 143.51 101.6 0)
-			(effects
-				(font
-					(size 1.27 1.27)
-				)
-				(justify right)
-			)
-		)
-		(pin "GPIO40" input
-			(at 143.51 104.14 0)
-			(effects
-				(font
-					(size 1.27 1.27)
-				)
-				(justify right)
-			)
-		)
-		(pin "GPIO37" input
-			(at 143.51 106.68 0)
-			(effects
-				(font
-					(size 1.27 1.27)
-				)
-				(justify right)
-			)
-		)
 		(pin "TX" input
 			(at 114.3 90.17 180)
@@
 			)
 		)
-		(pin "GPIO8" input
-			(at 114.3 118.11 180)
-			(effects
-				(font
-					(size 1.27 1.27)
-				)
-				(justify left)
-			)
-		)
-		(pin "GPIO6" input
-			(at 114.3 113.03 180)
-			(effects
-				(font
-					(size 1.27 1.27)
-				)
-				(justify left)
-			)
-		)
-		(pin "GPIO9" input
-			(at 114.3 120.65 180)
-			(effects
-				(font
-					(size 1.27 1.27)
-				)
-				(justify left)
-			)
-		)
-		(pin "GPIO11" input
-			(at 114.3 125.73 180)
-			(effects
-				(font
-					(size 1.27 1.27)
-				)
-				(justify left)
-			)
-		)
 		(pin "GPIO18" input
 			(at 114.3 138.43 180)
@@
 			(effects
 				(font
-					(size 1.27 1.27)
-				)
-				(justify left)
-			)
-		)
-		(pin "GPIO10" input
-			(at 114.3 123.19 180)
-			(effects
-				(font
