File: Fjernbetjening/Sender/PCB/CONTROL WIFI ESP32 S3 V4.0.kicad_pcb (KiCad board)
At the start: 4 copper layers, 90 x 60 mm, 45 parts, among them J1 Prog, J2 Bat, J3 USB_A, Q1 BC846BS, SW2 SW_Push, SW3 SW_Push, SW4 SW_Push, SW5 SW_Push, U1 USBLC6-2SC6, U2 MCP73832-2-OT, U4 COM-09032, U5 COM-09032, U6 CP2102N-Axx-xQFN28, U7 AP2112K-3.3, U8 ESP32-S2-WROVER

Commit message: mods on PCB done
Parts:
- removed BT3: SW_Push, Button_Switch_SMD:SW_Tactile_SPST_NO_Straight_CK_PTS636Sx25SMTRLFS
- removed C10: 0.1uf, Capacitor_SMD:C_0603_1608Metric
- removed SW5: SW_Push, Button_Switch_SMD:SW_SPST_PTS645
- removed U8: ESP32-S2-WROVER, RF_Module:ESP32-S2-WROVER
- added BT1: SW_Push, Button_Switch_SMD:SW_Tactile_SPST_NO_Straight_CK_PTS636Sx25SMTRLFS, F.Cu at (104.9, 123.8)
- added C9: 10u, Capacitor_SMD:C_0603_1608Metric, F.Cu at (62.5, 126.2)
- added SW1: SW_Push, Button_Switch_THT:SW_Tactile_SPST_Angled_PTS645Vx39-2LFS, F.Cu at (40.5, 84.1)
- added U3: USBLC6-2SC6, Package_TO_SOT_SMD:SOT-23-6, F.Cu at (59.3, 128.9)
- C1: value 0.1uf -> 1uF
- C2: value 100n -> 10nF
- C4: value 10u -> 1uF
- C5: value 10nF -> 0.1uf
- C6, C7, C8: value 1uF -> 0.1uf
- D1: value PWR ON -> Chrg
- D2: value Chrg -> PWR ON
- J1: value Prog -> USB_A; footprint Connector_PinHeader_1.27mm:PinHeader_2x03_P1.27mm_Vertical_SMD -> Connector_USB:USB_Mini-B_Wuerth_65100516121_Horizontal
- J3: value USB_A -> Prog; footprint Connector_USB:USB_Mini-B_Wuerth_65100516121_Horizontal -> Connector_PinHeader_1.27mm:PinHeader_2x03_P1.27mm_Vertical_SMD
- R1: value 330 -> 2k
- R10, R9: value 4.7k -> 10K
- R12: value 10k -> 4.7k
- R13: value 10k -> 1k
- R14: value 10K -> 10k
- R15: value 4.7k -> 10k
- R2: value 2k -> 330
- R3: value 4.7k -> 330
- R4: value 330 -> 4.7k
- R5: value 10K -> 4.7k
- R6: value 1k -> 4.7k
- SW3: footprint Button_Switch_THT:SW_Tactile_SPST_Angled_PTS645Vx39-2LFS -> Button_Switch_SMD:SW_SPST_PTS645
- U1: value USBLC6-2SC6 -> MCP73832-2-OT; footprint Package_TO_SOT_SMD:SOT-23-6 -> Package_TO_SOT_SMD:SOT-23-5
- U2: value MCP73832-2-OT -> AP2112K-3.3
- U4: value COM-09032 -> ESP32-WROOM-32; footprint GL_Diverse:POT-COM-09032 -> RF_Module:ESP32-WROOM-32
- U6: value CP2102N-Axx-xQFN28 -> COM-09032; footprint Package_DFN_QFN:QFN-28-1EP_5x5mm_P0.5mm_EP3.35x3.35mm -> GL_Diverse:POT-COM-09032
- U7: value AP2112K-3.3 -> CP2102N-Axx-xQFN28; footprint Package_TO_SOT_SMD:SOT-23-5 -> Package_DFN_QFN:QFN-28-1EP_5x5mm_P0.5mm_EP3.35x3.35mm
- moved R10 61.1 mm to (111.5, 122.2)
- moved J1 58.9 mm to (59.5, 135.6)
- moved R15 57.5 mm to (52.9, 124.2), turned to -90 degrees
- moved R12 55.9 mm to (101.9, 89.2)
- moved J3 54.7 mm to (89.4, 86.7)
- moved C1 54.7 mm to (72.8, 135.9), turned to 180 degrees
- moved C7 53.0 mm to (62.5, 82.6), turned to 180 degrees
- moved SW3 52.2 mm to (82.0, 111.7)
- moved R11 51.5 mm to (62.5, 90.7), turned to 180 degrees
- moved C6 50.0 mm to (62.5, 85.8), turned to 0 degrees
- moved U6 43.9 mm to (104.2, 105.0), turned to 0 degrees
- moved R4 43.0 mm to (111.4, 123.8)
- moved R14 41.8 mm to (55.2, 126.8)
- moved R5 37.5 mm to (36.4, 87.2)
- moved C5 37.2 mm to (111.4, 125.4)
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Connections:
- C1 pad 1: GND -> +5V
- C1 pad 2: EN -> GND
- C2 pad 1: GND -> VIN
- C2 pad 2: +3.3V -> GND
- C3 pad 1: GND -> Net-(U2-EN)
- C3 pad 2: +3.3V -> GND
- C5 pad 1: VIN -> BT
- C6 pad 1: Net-(U7-EN) -> GND
- C6 pad 2: GND -> EN
- C7 pad 1: +3.3V -> GND
- C7 pad 2: GND -> +3.3V
- C8 pad 1: +5V -> GND
- C8 pad 2: GND -> +3.3V
- D1 pad 1: GND -> Net-(D1-K)
- D2 pad 1: Net-(D2-K) -> GND
- FB1 pad 1: Net-(U7-EN) -> Net-(U2-EN)
- J1 pad 1: EN -> +5V
- J1 pad 2: +3.3V -> Net-(J1-D-)
- J1 pad 3: TX -> Net-(J1-D+)
- J1 pad 5: RX -> GND
- J1 pad 6: BT -> (no net)
- J3 pad 1: +5V -> EN
- J3 pad 2: Net-(J3-D-) -> +3.3V
- J3 pad 3: Net-(J3-D+) -> TX
- J3 pad 5: GND -> RX
- J3 pad 6: (no net) -> BT
- POT2 pad 2: IO6 -> IO4
- R1 pad 1: +3.3V -> Net-(U1-PROG)
- R1 pad 2: Net-(D1-A) -> GND
- R10 pad 2: IO12 -> BT
- R11 pad 1: +3.3V -> IO35
- R11 pad 2: IO9 -> +3.3V
- R12 pad 1: Net-(Q1A-B1) -> IO19
- R12 pad 2: Net-(Q1B-E2) -> +3.3V
- R13 pad 1: Net-(Q1B-B2) -> +3.3V
- R13 pad 2: Net-(Q1A-E1) -> Net-(U7-~{RST})
- R14 pad 1: +3.3V -> Net-(Q1A-B1)
- R14 pad 2: BT -> Net-(Q1B-E2)
- R15 pad 1: IO37 -> Net-(Q1B-B2)
- R15 pad 2: +3.3V -> Net-(Q1A-E1)
- R2 pad 1: Net-(U2-PROG) -> +5V
- R2 pad 2: GND -> Net-(D1-A)
- R3 pad 1: IO8 -> +3.3V
- R3 pad 2: +3.3V -> Net-(D2-A)
- R4 pad 1: +5V -> +3.3V
- R4 pad 2: Net-(D2-A) -> BT
- R5 pad 2: EN -> IO15
- R6 pad 2: Net-(U6-~{RST}) -> IO13
- R7 pad 2: BT -> IO12
- R8 pad 2: IO15 -> IO2
- R9 pad 2: IO13 -> EN
- SW2 pad 1: IO15 -> IO13
- SW3 pad 1: IO13 -> IO12
- SW4 pad 1: IO12 -> IO2
- U1 pad 1: Net-(J3-D-) -> Net-(D1-K)
- U1 pad 3: Net-(J3-D+) -> VIN
- U1 pad 4: USBN -> +5V
- U1 pad 5: +5V -> Net-(U1-PROG)
- U2 pad 1: Net-(D2-K) -> Net-(U2-EN)
- U2 pad 3: VIN -> Net-(U2-EN)
- U2 pad 4: +5V -> unconnected-(U2-NC-Pad4)
- U2 pad 5: Net-(U2-PROG) -> +3.3V
- U5 pad B1A: IO8 -> IO35
- U7 pad 1: Net-(U7-EN) -> unconnected-(U7-~{DCD}-Pad1)
- U7 pad 2: GND -> unconnected-(U7-~{RI}/CLK-Pad2)
- U7 pad 3: Net-(U7-EN) -> GND
- U7 pad 4: unconnected-(U7-NC-Pad4) -> USBP
- U7 pad 5: +3.3V -> USBN
Routing:
- net IO2: track 0.00 -> 63.9 mm
- net IO9: track 59.7 -> 0.00 mm
- net IO6: track 52.3 -> 0.00 mm, vias 2 -> 0
- net IO4: track 0.00 -> 41.4 mm, vias 0 -> 1
- net EN: track 60.8 -> 100.4 mm, vias 4 -> 2
- net IO14: track 0.00 -> 31.5 mm
- net IO16: track 0.00 -> 31.3 mm
- net IO37: track 29.3 -> 0.00 mm, vias 1 -> 0
- net IO38: track 28.7 -> 0.00 mm, vias 1 -> 0
- net IO8: track 21.7 -> 0.00 mm
- net IO19: track 0.00 -> 21.5 mm, vias 0 -> 1
- net IO12: track 51.7 -> 30.3 mm
- net IO35: track 0.00 -> 20.6 mm
- net IO15: track 57.0 -> 76.1 mm
- net IO40: track 15.6 -> 0.00 mm, vias 1 -> 0
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- removed copper zone on In2.Cu, net +3.3V
- removed copper zone on In1.Cu, net GND
Other:
- copper layers 4 -> 2
