File: Fjernbetjening/Sender/PCB/CONTROL WIFI ESP32 S3 V4.0.kicad_sch (KiCad schematic)
At the start: 28 parts, among them J2 Bat, J3 USB_A, SW2 SW_Push, SW3 SW_Push, SW4 SW_Push, SW5 SW_Push, U1 USBLC6-2SC6, U2 MCP73832-2-OT, U7 AP2112K-3.3

Commit message: mods on PCB done
Parts:
- renumbered C8 to C1, C5 to C2, C6 to C3, C7 to C4, D2 to D1, J3 to J1, R2 to R1, R4 to R2, R7 to R4, R8 to R5, R9 to R6, R10 to R7, R11 to R8, SW2 to SW1, SW3 to SW2, SW4 to SW3, SW5 to SW4, U2 to U1, U7 to U2, U1 to U3
Connections:
- net at J1.2 (D-): now also U3.3 (I/O2); no longer U3.1 (I/O1)
- net at J1.3 (D+): now also U3.1 (I/O1); no longer U3.3 (I/O2)
- net IO6 renamed IO4
- net IO9 renamed IO2
- no-connect marks 4 -> 1
Other:
- sheet STDEsp32: file StdEsp32.kicad_sch -> StdEsp32_worm2.kicad_sch
- sheet STDEsp32 ports: added GPIO14, GPIO16, GPIO19, GPIO21, GPIO22; removed GPIO10, GPIO11, GPIO3, GPIO37, GPIO38, GPIO40, GPIO6, GPIO7, GPIO8, GPIO9
