File: Fjernbetjening/Sender/PCB/Joystick.kicad_sch (KiCad schematic)
At the start: 2 parts, among them U4 COM-09032

Commit message: mods on PCB done
Parts:
- renumbered R15 to R11, U4 to U5
Changed lines of the file:
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@@
 		(on_board yes)
 		(dnp no)
-		(property "Reference" "U4"
+		(property "Reference" "U5"
 			(at 142.24 69.85 0)
 			(effects
@@
 			)
 		)
-		(property "Description" "\nJoystick, 2 - Axis Analog (Resistive) Output\n"
+		(property "Description" "Joystick, 2 - Axis Analog (Resistive) Output"
 			(at 148.59 90.17 0)
 			(effects
@@
 		(instances
 			(project "CONTROL WIFI ESP32 S3 V4.0"
-				(path "/a258bf7a-7e28-44d5-b6ba-b08ce88d15ec/6eda1525-bf1b-4dc6-873b-0e1de818b322"
-					(reference "U4")
-					(unit 1)
-				)
 				(path "/a258bf7a-7e28-44d5-b6ba-b08ce88d15ec/99cc5c98-6514-47dd-bb58-54f3159921a5"
 					(reference "U5")
+					(unit 1)
+				)
+				(path "/a258bf7a-7e28-44d5-b6ba-b08ce88d15ec/e07ae3a1-b9e3-40ea-b295-881946743af4"
+					(reference "U6")
 					(unit 1)
 				)
@@
 		(dnp no)
 		(fields_autoplaced yes)
-		(property "Reference" "#PWR021"
+		(property "Reference" "#PWR030"
 			(at 129.54 88.9 0)
 			(effects
@@
 		(instances
 			(project "CONTROL WIFI ESP32 S3 V4.0"
-				(path "/a258bf7a-7e28-44d5-b6ba-b08ce88d15ec/6eda1525-bf1b-4dc6-873b-0e1de818b322"
-					(reference "#PWR021")
-					(unit 1)
-				)
 				(path "/a258bf7a-7e28-44d5-b6ba-b08ce88d15ec/99cc5c98-6514-47dd-bb58-54f3159921a5"
-					(reference "#PWR014")
+					(reference "#PWR030")
+					(unit 1)
+				)
+				(path "/a258bf7a-7e28-44d5-b6ba-b08ce88d15ec/e07ae3a1-b9e3-40ea-b295-881946743af4"
+					(reference "#PWR036")
 					(unit 1)
 				)
@@
 		(dnp no)
 		(fields_autoplaced yes)
-		(property "Reference" "R15"
+		(property "Reference" "R11"
 			(at 108.458 96.5778 0)
 			(effects
@@
 		(instances
 			(project "CONTROL WIFI ESP32 S3 V4.0"
-				(path "/a258bf7a-7e28-44d5-b6ba-b08ce88d15ec/6eda1525-bf1b-4dc6-873b-0e1de818b322"
-					(reference "R15")
-					(unit 1)
-				)
 				(path "/a258bf7a-7e28-44d5-b6ba-b08ce88d15ec/99cc5c98-6514-47dd-bb58-54f3159921a5"
-					(reference "R3")
+					(reference "R11")
+					(unit 1)
+				)
+				(path "/a258bf7a-7e28-44d5-b6ba-b08ce88d15ec/e07ae3a1-b9e3-40ea-b295-881946743af4"
+					(reference "R12")
 					(unit 1)
 				)
@@
 		(dnp no)
 		(fields_autoplaced yes)
-		(property "Reference" "#PWR019"
+		(property "Reference" "#PWR029"
 			(at 128.27 116.84 0)
 			(effects
@@
 		(instances
 			(project "CONTROL WIFI ESP32 S3 V4.0"
-				(path "/a258bf7a-7e28-44d5-b6ba-b08ce88d15ec/6eda1525-bf1b-4dc6-873b-0e1de818b322"
-					(reference "#PWR019")
-					(unit 1)
-				)
 				(path "/a258bf7a-7e28-44d5-b6ba-b08ce88d15ec/99cc5c98-6514-47dd-bb58-54f3159921a5"
-					(reference "#PWR016")
+					(reference "#PWR029")
+					(unit 1)
+				)
+				(path "/a258bf7a-7e28-44d5-b6ba-b08ce88d15ec/e07ae3a1-b9e3-40ea-b295-881946743af4"
+					(reference "#PWR035")
 					(unit 1)
 				)
@@
 		(dnp no)
 		(fields_autoplaced yes)
-		(property "Reference" "#PWR022"
+		(property "Reference" "#PWR031"
 			(at 138.43 90.17 0)
 			(effects
@@
 		(instances
 			(project "CONTROL WIFI ESP32 S3 V4.0"
-				(path "/a258bf7a-7e28-44d5-b6ba-b08ce88d15ec/6eda1525-bf1b-4dc6-873b-0e1de818b322"
-					(reference "#PWR022")
-					(unit 1)
-				)
 				(path "/a258bf7a-7e28-44d5-b6ba-b08ce88d15ec/99cc5c98-6514-47dd-bb58-54f3159921a5"
-					(reference "#PWR012")
+					(reference "#PWR031")
+					(unit 1)
+				)
+				(path "/a258bf7a-7e28-44d5-b6ba-b08ce88d15ec/e07ae3a1-b9e3-40ea-b295-881946743af4"
+					(reference "#PWR037")
 					(unit 1)
 				)
@@
 		(dnp no)
 		(fields_autoplaced yes)
-		(property "Reference" "#PWR040"
+		(property "Reference" "#PWR032"
 			(at 139.7 80.01 0)
 			(effects
@@
 		(instances
 			(project "CONTROL WIFI ESP32 S3 V4.0"
-				(path "/a258bf7a-7e28-44d5-b6ba-b08ce88d15ec/6eda1525-bf1b-4dc6-873b-0e1de818b322"
-					(reference "#PWR040")
-					(unit 1)
-				)
 				(path "/a258bf7a-7e28-44d5-b6ba-b08ce88d15ec/99cc5c98-6514-47dd-bb58-54f3159921a5"
-					(reference "#PWR013")
+					(reference "#PWR032")
+					(unit 1)
+				)
+				(path "/a258bf7a-7e28-44d5-b6ba-b08ce88d15ec/e07ae3a1-b9e3-40ea-b295-881946743af4"
+					(reference "#PWR038")
 					(unit 1)
 				)
@@
 		(dnp no)
 		(fields_autoplaced yes)
-		(property "Reference" "#PWR018"
+		(property "Reference" "#PWR028"
 			(at 124.46 99.06 0)
 			(effects
@@
 		(instances
 			(project "CONTROL WIFI ESP32 S3 V4.0"
-				(path "/a258bf7a-7e28-44d5-b6ba-b08ce88d15ec/6eda1525-bf1b-4dc6-873b-0e1de818b322"
-					(reference "#PWR018")
-					(unit 1)
-				)
 				(path "/a258bf7a-7e28-44d5-b6ba-b08ce88d15ec/99cc5c98-6514-47dd-bb58-54f3159921a5"
-					(reference "#PWR015")
+					(reference "#PWR028")
+					(unit 1)
+				)
+				(path "/a258bf7a-7e28-44d5-b6ba-b08ce88d15ec/e07ae3a1-b9e3-40ea-b295-881946743af4"
+					(reference "#PWR034")
 					(unit 1)
 				)
@@
 		(dnp no)
 		(fields_autoplaced yes)
-		(property "Reference" "#PWR017"
+		(property "Reference" "#PWR027"
 			(at 106.68 97.79 0)
 			(effects
@@
 		(instances
 			(project "CONTROL WIFI ESP32 S3 V4.0"
-				(path "/a258bf7a-7e28-44d5-b6ba-b08ce88d15ec/6eda1525-bf1b-4dc6-873b-0e1de818b322"
-					(reference "#PWR017")
-					(unit 1)
-				)
 				(path "/a258bf7a-7e28-44d5-b6ba-b08ce88d15ec/99cc5c98-6514-47dd-bb58-54f3159921a5"
-					(reference "#PWR07")
-					(unit 1)
-				)
+					(reference "#PWR027")
+					(unit 1)
+				)
+				(path "/a258bf7a-7e28-44d5-b6ba-b08ce88d15ec/e07ae3a1-b9e3-40ea-b295-881946743af4"
+					(reference "#PWR033")
+					(unit 1)
+				)
