File: Fjernbetjening/Sender/PCB/USBSerial.kicad_sch (KiCad schematic)
At the start: 6 parts, among them Q1 BC846BS, U6 CP2102N-Axx-xQFN28

Commit message: mods on PCB done
Parts:
- renumbered C4 to C9, R6 to R13, R12 to R14, R13 to R15, U6 to U7
Changed lines of the file:
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@@
 		(dnp no)
 		(fields_autoplaced yes)
-		(property "Reference" "C4"
+		(property "Reference" "C9"
 			(at 93.7641 47.0541 0)
 			(effects
@@
 			(project "CONTROL WIFI ESP32 S3 V4.0"
 				(path "/a258bf7a-7e28-44d5-b6ba-b08ce88d15ec/949b0c8e-834d-483d-a031-0a34e77ac93c"
-					(reference "C4")
+					(reference "C9")
 					(unit 1)
 				)
@@
 		(dnp no)
 		(fields_autoplaced yes)
-		(property "Reference" "#PWR028"
+		(property "Reference" "#PWR041"
 			(at 91.44 57.15 0)
 			(effects
@@
 			(project "CONTROL WIFI ESP32 S3 V4.0"
 				(path "/a258bf7a-7e28-44d5-b6ba-b08ce88d15ec/949b0c8e-834d-483d-a031-0a34e77ac93c"
-					(reference "#PWR028")
+					(reference "#PWR041")
 					(unit 1)
 				)
@@
 		(dnp no)
 		(fields_autoplaced yes)
-		(property "Reference" "#PWR031"
+		(property "Reference" "#PWR039"
 			(at 64.77 49.53 0)
 			(effects
@@
 			(project "CONTROL WIFI ESP32 S3 V4.0"
 				(path "/a258bf7a-7e28-44d5-b6ba-b08ce88d15ec/949b0c8e-834d-483d-a031-0a34e77ac93c"
-					(reference "#PWR031")
+					(reference "#PWR039")
 					(unit 1)
 				)
@@
 		(on_board yes)
 		(dnp no)
-		(property "Reference" "R12"
+		(property "Reference" "R14"
 			(at 128.27 55.9816 90)
 			(effects
@@
 			(project "CONTROL WIFI ESP32 S3 V4.0"
 				(path "/a258bf7a-7e28-44d5-b6ba-b08ce88d15ec/949b0c8e-834d-483d-a031-0a34e77ac93c"
-					(reference "R12")
+					(reference "R14")
 					(unit 1)
 				)
@@
 		(dnp no)
 		(fields_autoplaced yes)
-		(property "Reference" "U6"
+		(property "Reference" "U7"
 			(at 87.2841 121.1001 0)
 			(effects
@@
 			(project "CONTROL WIFI ESP32 S3 V4.0"
 				(path "/a258bf7a-7e28-44d5-b6ba-b08ce88d15ec/949b0c8e-834d-483d-a031-0a34e77ac93c"
-					(reference "U6")
+					(reference "U7")
 					(unit 1)
 				)
@@
 		(on_board yes)
 		(dnp no)
-		(property "Reference" "R13"
+		(property "Reference" "R15"
 			(at 128.27 69.9516 90)
 			(effects
@@
 			(project "CONTROL WIFI ESP32 S3 V4.0"
 				(path "/a258bf7a-7e28-44d5-b6ba-b08ce88d15ec/949b0c8e-834d-483d-a031-0a34e77ac93c"
-					(reference "R13")
+					(reference "R15")
 					(unit 1)
 				)
@@
 		(dnp no)
 		(fields_autoplaced yes)
-		(property "Reference" "#PWR030"
+		(property "Reference" "#PWR042"
 			(at 104.14 86.36 0)
 			(effects
@@
 			(project "CONTROL WIFI ESP32 S3 V4.0"
 				(path "/a258bf7a-7e28-44d5-b6ba-b08ce88d15ec/949b0c8e-834d-483d-a031-0a34e77ac93c"
-					(reference "#PWR030")
+					(reference "#PWR042")
 					(unit 1)
 				)
@@
 		(dnp no)
 		(fields_autoplaced yes)
-		(property "Reference" "#PWR024"
+		(property "Reference" "#PWR040"
 			(at 85.09 128.27 0)
 			(effects
@@
 			(project "CONTROL WIFI ESP32 S3 V4.0"
 				(path "/a258bf7a-7e28-44d5-b6ba-b08ce88d15ec/949b0c8e-834d-483d-a031-0a34e77ac93c"
-					(reference "#PWR024")
+					(reference "#PWR040")
 					(unit 1)
 				)
@@
 		(dnp no)
 		(fields_autoplaced yes)
-		(property "Reference" "R6"
+		(property "Reference" "R13"
 			(at 66.548 55.9378 0)
 			(effects
@@
 			(project "CONTROL WIFI ESP32 S3 V4.0"
 				(path "/a258bf7a-7e28-44d5-b6ba-b08ce88d15ec/949b0c8e-834d-483d-a031-0a34e77ac93c"
-					(reference "R6")
-					(unit 1)
-				)
+					(reference "R13")
+					(unit 1)
+				)
