File: Fjernbetjening/Modtager/Lys.kicad_sch (KiCad schematic)
At the start: 15 parts, among them J4 Conn_01x02, J5 Conn_01x02, Q2 AO3400A, Q3 AO3400A, Q4 AO3400A

Commit message: forberedelse for drone
Parts:
- added R10, R11, R19: 10K, Resistor_SMD:R_0603_1608Metric, symbol Device:R
Connections:
- net AgterLys: now also R11.1
- net GND: now also R10.2, R11.2, R19.2
- net KabineLys: now also R19.1
- net Lanterne: now also R10.1
