File: Fjernbetjening/Modtager/StdEsp32_worm2.kicad_sch (KiCad schematic)
At the start: 7 parts, among them J1 Prog, U3 ESP32-WROOM-32

Commit message: forberedelse for drone
Parts:
- added R14, R15: 10K, Resistor_SMD:R_0603_1608Metric, symbol Device:R
Connections:
- net +3.3V: now also R14.1, R15.2
- net SCL: now reaches U3.36 (IO22)
- net SCL: now also R14.2
- net SDA: now reaches U3.37 (IO23)
- net SDA: now also R15.1
