File: Fjernbetjening/Modtager/TocBoatReceiver.kicad_pcb (KiCad board)
At the start: 2 copper layers, 55 x 85 mm, 40 parts, among them J1 Prog, J2 USB_A, J3 Battery, J4 Conn_01x02, J5 Conn_01x02, J6 SpeedController, J7 Servo, Q1 BC846BS, Q2 AO3400A, Q3 AO3400A, Q4 AO3400A, U1 USBLC6-2SC6, U2 AP1117-33, U3 ESP32-WROOM-32, U6 CP2102N-Axx-xQFN28

Commit message: update
Routing:
- net Net-(D4-A): track 0.00 -> 3.12 mm
- net Net-(D2-A): track 0.00 -> 2.03 mm
Changed lines of the file:
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@@
+	)
+	(segment
+		(start 183.9375 130.0625)
+		(end 184 130)
+		(width 0.2)
+		(layer "F.Cu")
+		(net 7)
+	)
+	(segment
+		(start 183.9375 132)
+		(end 183.9375 130.0625)
+		(width 0.2)
+		(layer "F.Cu")
+		(net 7)
 	)
 	(segment
@@
 	)
 	(segment
+		(start 184.65 52.2875)
+		(end 184.9375 52)
+		(width 0.2)
+		(layer "F.Cu")
+		(net 9)
+	)
+	(segment
+		(start 184.65 55)
+		(end 184.65 52.2875)
+		(width 0.2)
+		(layer "F.Cu")
+		(net 9)
+	)
+	(segment

Commit message: forberedelse for drone
Parts:
- removed C8: 0.1uf, Capacitor_SMD:C_0603_1608Metric
- added D5: BZT52B-C20, Diode_SMD:D_SOD-123F, F.Cu at (172.8, 110.0)
- added D6: BZT52B-C20, Diode_SMD:D_SOD-123F, F.Cu at (172.4, 100.0)
- added J8: PowerESC, Connector_Molex:Molex_KK-254_AE-6410-02A_1x02_P2.54mm_Vertical, F.Cu at (173.0, 72.5)
- added R14: 10K, Resistor_SMD:R_0603_1608Metric, F.Cu at (165.3, 102.5)
- added R15: 10K, Resistor_SMD:R_0603_1608Metric, F.Cu at (165.2, 100.5)
- added R16: 100, Resistor_SMD:R_0603_1608Metric, F.Cu at (174.5, 108.0)
- added R17: 0.01R, Resistor_SMD:R_1812_4532Metric, F.Cu at (178.0, 106.4)
- added R18: 100, Resistor_SMD:R_0603_1608Metric, F.Cu at (174.5, 105.5)
- added R19: 10K, Resistor_SMD:R_0603_1608Metric, F.Cu at (157.0, 96.8)
- added U4: SAM-M8Q, RF_GPS:ublox_SAM-M8Q, F.Cu at (144.9, 64.1)
- added U5: INA219BxD, Package_SO:SOIC-8_3.9x4.9mm_P1.27mm, F.Cu at (170.1, 105.0)
- moved R10 25.4 mm to (159.8, 86.0)
- moved R11 23.3 mm to (157.0, 92.7), turned to -90 degrees
- moved R6 0.10 mm to (149.6, 125.0)
Connections:
- C7 pad 1: +BATT -> Net-(J3-Pin_1)
- J3 pad 1: +BATT -> Net-(J3-Pin_1)
- J6 pad 2: /ESP32/GPIO16 -> /ESP32/GPIO4
- Q2 pad 1: /ESP32/GPIO15 -> /ESP32/GPIO12
- Q3 pad 1: /ESP32/GPIO17 -> /ESP32/GPIO13
- Q4 pad 1: /ESP32/GPIO18 -> /ESP32/GPIO15
- R10 pad 1: +BATT -> /ESP32/GPIO15
- R10 pad 2: /ESP32/GPIO5 -> GND
- R11 pad 1: /ESP32/GPIO5 -> /ESP32/GPIO13
- U3 pad 36: unconnected-(U3-IO22-Pad36) -> /ESP32/SCL
- U3 pad 37: unconnected-(U3-IO23-Pad37) -> /ESP32/SDA
Routing:
- net +3.3V: track 118.0 -> 44.0 mm, vias 7 -> 11
- net GND: track 26.0 -> 95.2 mm, vias 51 -> 3
- net /ESP32/GPIO5: track 51.0 -> 0.00 mm
- net /ESP32/SDA: track 0.00 -> 48.0 mm
- net /ESP32/SCL: track 0.00 -> 47.3 mm, vias 0 -> 2
- net /ESP32/GPIO16: track 49.2 -> 8.88 mm, vias 0 -> 2
- net /ESP32/GPIO4: track 0.00 -> 38.2 mm, vias 0 -> 1
- net /ESP32/GPIO18: track 28.4 -> 0.00 mm
- net Net-(J3-Pin_1): track 0.00 -> 26.5 mm
- net /ESP32/GPIO17: track 27.8 -> 8.88 mm
- net /ESP32/GPIO12: track 0.00 -> 10.2 mm
- net Net-(D6-K): track 0.00 -> 9.90 mm
- net /ESP32/GPIO13: track 0.00 -> 8.91 mm
- net /ESP32/GPIO15: track 19.5 -> 12.0 mm
- net /ESP32/GPIO14: track 49.1 -> 54.7 mm, vias 4 -> 2
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- added copper zone on B.Cu, net +3.3V
- removed copper zone on B.Cu, net GND
