File: Fjernbetjening/Modtager/_autosave-TocBoatReceiver.kicad_sch (KiCad schematic)
At the start: 17 parts, among them J2 USB_A, J3 Battery, J6 SpeedController, J7 Servo, J8 PowerESC, U1 USBLC6-2SC6, U2 AP1117-33, U4 SAM-M8Q, U5 INA219BxD

Commit message: forberedelse for drone
Connections:
- net ESP32/GPIO16: no longer J6.2 (Pin_2)
- net ESP32/GPIO4: now also J6.2 (Pin_2)
Changed lines of the file:
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@@
 	(wire
 		(pts
+			(xy 149.86 111.76) (xy 143.51 111.76)
+		)
+		(stroke
+			(width 0)
+			(type default)
+		)
+	)
+	(wire
+		(pts
 			(xy 176.53 55.88) (xy 194.31 55.88)
 		)
@@
 	(wire
 		(pts
+			(xy 149.86 111.76) (xy 149.86 118.11)
+		)
+		(stroke
+			(width 0)
+			(type default)
+		)
+	)
+	(wire
+		(pts
 			(xy 104.14 133.35) (xy 114.3 133.35)
 		)
@@
 	(wire
 		(pts
-			(xy 143.51 119.38) (xy 149.86 119.38)
-		)
-		(stroke
-			(width 0)
-			(type default)
-		)
-	)
-	(wire
-		(pts
 			(xy 95.25 59.69) (xy 97.79 59.69)
 		)
@@
 	(wire
 		(pts
-			(xy 149.86 119.38) (xy 149.86 118.11)
-		)
-		(stroke
-			(width 0)
-			(type default)
-		)
-	)
-	(wire
-		(pts
 			(xy 143.51 105.41) (xy 199.39 105.41)
 		)
@@
 		)
 		(pin "GPIO4" input
-			(at 114.3 107.95 180)
+			(at 143.51 111.76 0)
 			(effects
 				(font
 					(size 1.27 1.27)
 				)
-				(justify left)
+				(justify right)
 			)
 		)
@@
 		)
 		(pin "GPIO18" input
-			(at 114.3 138.43 180)
+			(at 143.51 114.3 0)
 			(effects
 				(font
 					(size 1.27 1.27)
 				)
-				(justify left)
+				(justify right)
 			)
 		)
@@
 		)
 		(pin "GPIO17" input
-			(at 114.3 135.89 180)
+			(at 143.51 116.84 0)
 			(effects
 				(font
 					(size 1.27 1.27)
 				)
-				(justify left)
+				(justify right)
 			)
 		)
