File: Fjernbetjening/Sender/RcSender.kicad_pcb (KiCad board)
At the start: 2 copper layers, 90 x 60 mm, 45 parts, among them J1 USB_A, J2 Bat, J3 Prog, Q1 BC846BS, SW1 SW_Push, SW2 SW_Push, SW3 SW_Push, SW4 SW_Push, U1 MCP73832-2-OT, U2 AP2112K-3.3, U3 USBLC6-2SC6, U4 ESP32-WROOM-32, U5 COM-09032, U6 COM-09032, U7 CP2102N-Axx-xQFN28

Commit message: forberedelse for drone
Parts:
- BT1: footprint Button_Switch_SMD:SW_Tactile_SPST_NO_Straight_CK_PTS636Sx25SMTRLFS -> Button_Switch_SMD:SW_SPST_PTS645
- moved R7 20.8 mm to (85.8, 128.0)
- moved SW3 12.1 mm to (82.0, 123.8)
- moved J2 1.10 mm to (78.0, 140.0)
- moved BT1 0.44 mm to (104.5, 123.8)
Connections:
- R7 pad 1: +3.3V -> IO12
- R7 pad 2: IO12 -> GND
- R8 pad 1: +3.3V -> IO2
- R8 pad 2: IO2 -> GND
- SW3 pad 1: IO12 -> +3.3V
- SW3 pad 2: GND -> IO12
- SW4 pad 1: IO2 -> +3.3V
- SW4 pad 2: GND -> IO2
Routing:
- net +3.3V: track 17.2 -> 43.2 mm, vias 15 -> 17
- net GND: track 15.5 -> 37.3 mm, vias 0 -> 1
- net IO12: track 30.3 -> 42.1 mm
- net BT: track 99.5 -> 110.7 mm, vias 2 -> 3
- net IO2: track 63.9 -> 58.6 mm, vias 0 -> 2
- net EN: track 100.4 -> 98.0 mm
- net VIN: track 16.6 -> 17.7 mm
