File: Fjernbetjening/Sender/RcSender.kicad_sch (KiCad schematic)
At the start: 28 parts, among them J1 USB_A, J2 Bat, SW1 SW_Push, SW2 SW_Push, SW3 SW_Push, SW4 SW_Push, U1 MCP73832-2-OT, U2 AP2112K-3.3, U3 USBLC6-2SC6

Commit message: forberedelse for drone
Parts:
- BT1: renamed from BT?; footprint Button_Switch_SMD:SW_Tactile_SPST_NO_Straight_CK_PTS636Sx25SMTRLFS -> Button_Switch_SMD:SW_SPST_PTS645
- gave numbers to parts that had none: 3
Connections:
- net +3.3V: now also SW3.1, SW4.1; no longer R7.1, R8.1
- net GND: now also R7.2, R8.2; no longer SW3.2, SW4.2
- net IO12: now also R7.1, SW3.2; no longer R7.2, SW3.1
- net IO2: now also R8.1, SW4.2; no longer R8.2, SW4.1
- no-connect marks 1 -> 10
Other:
- sheet STDEsp32 ports: added GPIO23, GPIO25, GPIO26, GPIO27, GPIO32, GPIO33, GPIO34; removed none
- moved on the sheet: R7, R8, SW3, SW4
